File: hw/indego_adapter.brd (EAGLE design)
At the start: 60 x 230 mm, 108 parts, among them Q1 IRF9530, Q3 IRLML2244

Commit message: new kicad pcb added
Parts:
- removed DC_5.5V1, DC_VIN: (no value), wirepad:2,54/1,0
- removed J_OLED3, J_OLED4: (no value), jumper:SJ_2
- removed OLED1: (no value), con-lstb:MA04-1
- removed PAD26, PAD27, PAD28, PAD29, PAD30, PAD31, PAD32, PAD33, PAD34, PAD35, PAD36, PAD37, PAD38, PAD39, PAD40, PAD41: (no value), wirepad:2,15/1,0
- removed PAD_GNDA, PAD_MLP, PAD_MLR, PAD_MRN, PAD_MRP: (no value), wirepad:3,17/1,3
- removed R1, R2: (no value), rcl:M0805
- removed RTC1: (no value), con-lstb:MA05-1
- removed SJ1: (no value), jumper:SJ
- removed SV2: (no value), con-ml:ML6
- removed SV3: (no value), con-ml:ML10
- added BUS_1: I2CBUS, con-amp-micromatch:MICROMATCH-10SMD
- added C4: (no value), rcl:C0805
- added C5: 0.47, rcl:C0805
- added C6, C7: 100n, rcl:C0805
- added DC_GND3, DC_GND4, DC_VIN1, DC_VIN2, U55SW, VCC: (no value), wirepad:2,54/1,0
- added GPS2, RTC: (no value), con-lstb:MA05-1
- added IC1: MEGA128-A, atmel:TQFP64
- added JP1: AVR-ISP-6VERT, avr-7:AVR-ISP-6
- added JP2: AVR-JTAG-10, avr-7:AVR-JTAG-10
- added J_UBSW, J_UBSW1: (no value), SparkFun-Jumpers:SMT-JUMPER_2_NO_NO-SILK
- added OLED: (no value), con-lstb:MA04-1
- added P_BUS_FON, P_BUS_INT, P_BUS_RESET, P_BUS_SCL, P_BUS_SDA, P_GND2, P_U5SW, P_UBSW, P_UBUS: (no value), wirepad:2,15/1,0
- added Q2: IRF9530, transistor-fet:TO220
- added R10, R11, R12, R13, R14, R15, R16, R8, R9: 100k, rcl:M0805
- added R17: 1, rcl:M0805
- added R18: 220k, rcl:R0805
- added R19, R23: 100k, rcl:R0805
- added R25: 0.1, rcl:R2512
- added SJGND, SJGND1: (no value), jumper:SJ
- added SV5: BNO055, con-lstb:MA08-1
- added T2: (no value), transistor:SOT23-BEC
- added TP1, TP10, TP11, TP12, TP13, TP14, TP15, TP2, TP3, TP4, TP5, TP6, TP7, TP8, TP9: TPB2,54, testpad:B2,54
- added U$2, U$4: 1X10, headers(2mm):1X10
- C2, C3: value (none) -> 100n
- F3: value FUSE 6A -> 10AT
- R5: value 10k -> 220k
- R6, R7: value 10k -> 100k
- SV1: device con-ml:ML10 -> con-lsta:FE13-2
- moved DC_GND2 76.2 mm to (14.0, 55.9), turned to 90 degrees
- moved DC_GND1 63.2 mm to (29.2, 55.9), turned to 90 degrees
- moved PAD23 55.9 mm to (35.6, 50.8)
- moved PAD19 55.9 mm to (35.6, 61.0)
- moved PAD21 55.9 mm to (35.6, 55.9)
- moved PAD24 55.9 mm to (35.6, 48.3)
- moved PAD18 55.9 mm to (35.6, 63.5)
- moved PAD20 55.9 mm to (35.6, 58.4)
- moved PAD22 55.9 mm to (35.6, 53.3)
- moved PAD25 55.9 mm to (35.6, 45.7)
- moved J_RPIVCC 52.9 mm to (34.7, 65.4), turned to 225 degrees
- moved SV1 44.4 mm to (34.3, 81.3), flipped to the bottom
- moved R4 39.4 mm to (25.4, 11.4), flipped to the bottom
- moved T1 36.7 mm to (22.9, 14.0), flipped to the bottom
- moved R3 34.9 mm to (26.7, 16.5), flipped to the bottom
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- renumbered PAD1 to P_ML_OUTA, PAD10 to P_UBSW2, PAD11 to P_GND1, PAD2 to P_ML_OUTB, PAD5 to P_MR_OUTA, PAD6 to P_MR_OUTB, PAD7 to P_MM_OUTA, PAD8 to P_MM_OUTB, PAD9 to P_UBSW1
Connections:
- removed net LCD_3: J_OLED3.2, OLED1.1
- removed net LCD_4: J_OLED4.2, OLED1.2
- removed net MOW_MOTOR_BLACK: U$3.P$24
- removed net MOW_MOTOR_RED: U$3.P$25
- removed net N$35: R2.1, SV1.8
- removed net N$36: R1.1, SV1.10
- removed net N$37: R20.2, RTC1.2, SV1.3
- removed net N$39: R22.2, RTC1.4, SV1.7
- removed net U5SW: PAD29.1, R.4, SV3.4, U$3.P$20
- removed net UCHARGE_N: U$3.P$3
- removed net UCHARGE_P: U$3.P$2
- removed net VCC_RPI: J_RPIVCC.1, RTC1.1, SV1.1
- new net AVCC: IC1.64
- new net BNO055_ADD: R15.2, R8.1, SV5.4
- new net BNO055_BOOT: R10.1, R13.2, SV5.2
- new net BNO055_INT: R14.2, R9.1, SV5.3
- new net BNO055_RESET: R11.1, R12.2, SV5.1
- new net BUS_UB: J_UBSW1.2, R.5
- new net BUS_UBSW: BUS_1.6, DC_VIN1.1, DC_VIN2.1, J_UBSW.2
- new net CHON: R23.2
- new net GPS_PPS: GPS2.5
- new net GPS_RXD: GPS2.4, U$4.8
- new net GPS_TXD: GPS2.3, U$4.9
- new net GPS_VCC: C5.1, GPS2.1, R17.2, U$4.10
- new net N$2: TP1.TP, U$2.2
- new net N$24: C4.2, R10.2, R11.2, R16.2, R8.2, R9.2, SV5.8
- new net N$25: TP2.TP, U$2.3
- new net N$26: TP3.TP, U$2.4
- new net N$27: TP4.TP, U$2.5
- new net N$29: TP5.TP, U$2.6
- new net N$3: Q2.1, R18.2, T2.C
- new net N$33: TP6.TP, U$2.7
- new net N$34: TP7.TP, U$2.8
- new net N$42: TP8.TP, U$2.9
- new net N$43: TP9.TP, U$2.10
- new net N$44: TP10.TP, U$4.2
- new net N$45: TP11.TP, U$4.3
- new net N$46: TP12.TP, U$4.4
- new net N$47: TP13.TP, U$4.5
- new net N$50: TP14.TP, U$4.6
- new net N$51: TP15.TP, U$4.7
- new net N$52: JP1.5
- new net N$53: JP1.3
- new net N$54: JP1.1
- new net N$55: JP1.4
- new net N$56: JP2.8
- new net N$57: JP2.6
- new net N$58: JP2.4
- new net N$59: JP2.7
- new net N$60: JP2.9
- new net N$61: JP2.3
- new net N$62: JP2.5
- new net N$63: JP2.1
- new net N$65: R19.2, R23.1, T2.B
- new net PGND: D2.A, MD_GND.1, PAD12.1, P_GND1.1, SJGND.2, SJGND1.2, U$1.P$24, U$1.P$25, U$3.P$3
- new net RPI_GPIO17: SV1.11
- new net RPI_GPIO18: SV1.12
- new net RPI_GPIO22: SV1.15
- new net RPI_GPIO23: SV1.16
- new net RPI_GPIO24: SV1.18
- new net RPI_GPIO25: SV1.22
- new net RPI_GPIO27: SV1.13
- new net RPI_INT: R22.2, RTC.4, SV1.7
- new net RPI_SCL: R21.2, RTC.3, SV1.5
- new net RPI_SDA: R20.2, RTC.2, SV1.3
- new net RPI_SPI0_CE0: SV1.24
- new net RPI_SPI0_CE1: SV1.26
- new net RPI_SPI0_MISO: SV1.21
- new net RPI_SPI0_MOSI: SV1.19
- new net RPI_SPI0_SCL: SV1.23
- new net RPI_VCC: J_RPIVCC.1, RTC.1, SV1.1, SV1.17
- new net UB_: C7.2, Q2.2, R25.1
- new net UCH: C6.2, Q2.3, R18.1, U$3.P$2
- net BUS_FON: now also BUS_1.3, P_BUS_FON.1; no longer PAD28.1, SV3.3
- net BUS_INT: now also BUS_1.9, P_BUS_INT.1; no longer PAD34.1, SV2.1, SV3.9
- net BUS_RESET: now also BUS_1.5, P_BUS_RESET.1; no longer PAD30.1, PAD40.1, SV2.5, SV3.5
- net BUS_SCL: now also BUS_1.7, P_BUS_SCL.1; no longer PAD32.1, PAD38.1, SV2.3, SV3.7
- net BUS_SDA: now also BUS_1.1, P_BUS_SDA.1; no longer PAD26.1, PAD36.1, PAD39.1, SV2.4, SV3.1
- net GND: now also BUS_1.10, BUS_1.8, C4.1, C5.2, DC_GND4.1, GPS2.2, IC1.22, IC1.53, IC1.63, JP1.6, JP2.10, JP2.2, OLED.1, P_GND2.1, R12.1, R13.1, R14.1, R15.1, RTC.5, SJGND1.1, SV5.7, U$2.1, U$4.1; no longer J_OLED3.1, J_OLED4.1, PAD33.1, PAD35.1, PAD41.1, RTC1.5, SJ1.2, SV1.9, SV2.6, SV3.10, SV3.8
- net GNDA: now also C6.1, C7.1, DC_GND3.1, R19.1, SJGND.1, SV1.14, SV1.20, SV1.25, SV1.9, T2.E; no longer D2.A, MD_GND.1, PAD_GNDA.1, SJ1.1, U$1.P$24, U$1.P$25
- net ML_OUTA: now also P_ML_OUTA.1; no longer PAD_MLP.1
- net ML_OUTB: now also P_ML_OUTB.1; no longer PAD_MLR.1
- net MM_OUTA: now also P_MM_OUTA.1, U$3.P$25
- net MM_OUTB: now also P_MM_OUTB.1, U$3.P$24
- net MR_OUTA: now also P_MR_OUTA.1; no longer PAD_MRP.1
- net MR_OUTB: now also P_MR_OUTB.1; no longer PAD_MRN.1
- net N$38: now also PAD13.1; no longer R21.2, RTC1.3, SV1.5
- net OLED_SCL: now also OLED.3; no longer OLED1.3
- net OLED_SDA: now also OLED.4; no longer OLED1.4
- net RPI_RXD: now also SV1.10; no longer R1.2
- net RPI_TXD: now also SV1.8; no longer R2.2
- net SCL_SCK: now also SV5.6
- net SDA_MOSI: now also SV5.5
- net U55SW: now also BUS_1.4, P_U5SW.1, R.4, U$3.P$20, U55SW.1; no longer DC_5.5V1.1
- net UB: now also J_UBSW1.1, R25.2; no longer R.5
- net UBSW: now also J_UBSW.1, P_UBSW.1, P_UBSW1.1, P_UBSW2.1; no longer DC_VIN.1, PAD31.1, SV3.6
- net UBUS: now also BUS_1.2, P_UBUS.1; no longer PAD27.1, PAD37.1, SV2.2, SV3.2
- net VCC: now also IC1.21, IC1.52, OLED.2, R16.1, R17.1, VCC.1; no longer J_OLED3.3, J_OLED4.3
Other:
- board size 60 x 230 mm -> 76.2 x 230 mm
- board text added: "simpleRTK2Blite"
