File: hw/indego_adapter.sch (EAGLE design)
At the start: 108 parts, among them Q1 IRF9530, Q3 IRLML2244

Commit message: new kicad pcb added
Parts:
- removed J_OLED3, J_OLED4: (no value), jumper:SJ2W
- removed OLED1: (no value), con-lstb:MA04-1
- removed PAD1, PAD10, PAD11, PAD2, PAD26, PAD27, PAD28, PAD29, PAD30, PAD31, PAD32, PAD33, PAD34, PAD35, PAD36, PAD37, PAD38, PAD39, PAD40, PAD41, PAD5, PAD6, PAD7, PAD8, PAD9: (no value), wirepad:2,15/1,0
- removed PAD_GNDA, PAD_MLP, PAD_MLR, PAD_MRN, PAD_MRP: (no value), wirepad:3,17/1,3
- removed R1, R2: (no value), rcl:R-EU_M0805
- removed SJ1: (no value), jumper:SJ
- removed SV2: (no value), con-ml:ML6
- removed SV3: (no value), con-ml:ML10
- added BUS_1: I2CBUS, con-amp-micromatch:MICROMATCH-10SMD
- added C4: (no value), rcl:C-EUC0805
- added C5: 0.47, rcl:C-EUC0805
- added C6, C7: 100n, rcl:C-EUC0805
- added DC_GND3, DC_GND4, DC_VIN2, VCC: (no value), wirepad:2,54/1,0
- added GPS2: (no value), con-lstb:MA05-1
- added IC1: MEGA128-A, atmel:MEGA128-A
- added JP1: AVR-ISP-6VERT, avr-7:AVR-ISP-6VERT
- added JP2: AVR-JTAG-10, avr-7:AVR-JTAG-10
- added J_UBSW, J_UBSW1: JUMPER-SMT_2_NO_NO-SILK, SparkFun-Jumpers:JUMPER-SMT_2_NO_NO-SILK
- added OLED: (no value), con-lstb:MA04-1
- added P_BUS_FON, P_BUS_INT, P_BUS_RESET, P_BUS_SCL, P_BUS_SDA, P_GND1, P_GND2, P_ML_OUTA, P_ML_OUTB, P_MM_OUTA, P_MM_OUTB, P_MR_OUTA, P_MR_OUTB, P_U5SW, P_UBSW, P_UBSW1, P_UBSW2, P_UBUS: (no value), wirepad:2,15/1,0
- added Q2: IRF9530, transistor-fet:IRF9530
- added R10, R11, R12, R13, R14, R15, R16, R8, R9: 100k, rcl:R-EU_M0805
- added R17: 1, rcl:R-EU_M0805
- added R18: 220k, rcl:R-EU_R0805
- added R19, R23: 100k, rcl:R-EU_R0805
- added R25: 0.1, rcl:R-EU_R2512
- added SJGND, SJGND1: (no value), jumper:SJ
- added SV5: BNO055, con-lstb:MA08-1
- added T2: (no value), transistor:BC817-16-NPN-SOT23-BEC
- added TP1, TP10, TP11, TP12, TP13, TP14, TP15, TP2, TP3, TP4, TP5, TP6, TP7, TP8, TP9: TPB2,54, testpad:TPB2,54
- added U$2, U$4: 1X10, headers(2mm):1X10
- C2, C3: value (none) -> 100n
- F3: value FUSE 6A -> 10AT
- R5: value 10k -> 220k
- R6, R7: value 10k -> 100k
- SV1: device con-ml:ML10 -> con-lsta:FE13-2
- renumbered DC_5.5V1 to U55SW, DC_VIN to DC_VIN1, RTC1 to RTC
Connections:
- net N$37 renamed RPI_SDA
- net N$38 renamed RPI_SCL
- net N$39 renamed RPI_INT
- removed net LCD_3: J_OLED3.2, OLED1.1
- removed net LCD_4: J_OLED4.2, OLED1.2
- removed net MOW_MOTOR_BLACK: U$3.P$23
- removed net MOW_MOTOR_RED: U$3.P$24
- removed net N$35: R2.1, SV1.8
- removed net N$36: R1.1, SV1.10
- removed net U5SW: PAD29.P, R.4, SV3.4, U$3.P$19
- removed net UCHARGE_N: U$3.P$2
- removed net UCHARGE_P: U$3.P$1
- removed net VCC_RPI: J_RPIVCC.1, RTC.1, SV1.1
- new net BNO055_ADD: R15.2, R8.1, SV5.4
- new net BNO055_BOOT: R10.1, R13.2, SV5.2
- new net BNO055_INT: R14.2, R9.1, SV5.3
- new net BNO055_RESET: R11.1, R12.2, SV5.1
- new net BUS_UB: J_UBSW1.2, R.5
- new net BUS_UBSW: BUS_1-6.S, DC_VIN1.P, DC_VIN2.P, J_UBSW.2
- new net CHON: R23.2
- new net GPS_PPS: GPS2.5
- new net GPS_RXD: GPS2.4, U$4.8
- new net GPS_TXD: GPS2.3, U$4.9
- new net GPS_VCC: C5.1, GPS2.1, R17.2, U$4.10
- new net N$2: TP1.TP, U$2.2
- new net N$24: C4.2, R10.2, R11.2, R16.2, R8.2, R9.2, SV5.8
- new net N$25: TP2.TP, U$2.3
- new net N$26: TP3.TP, U$2.4
- new net N$27: TP4.TP, U$2.5
- new net N$29: TP5.TP, U$2.6
- new net N$3: Q2.G, R18.2, T2.C
- new net N$33: TP6.TP, U$2.7
- new net N$34: TP7.TP, U$2.8
- new net N$38: PAD13.P
- new net N$42: TP8.TP, U$2.9
- new net N$43: TP9.TP, U$2.10
- new net N$44: TP10.TP, U$4.2
- new net N$45: TP11.TP, U$4.3
- new net N$46: TP12.TP, U$4.4
- new net N$47: TP13.TP, U$4.5
- new net N$50: TP14.TP, U$4.6
- new net N$51: TP15.TP, U$4.7
- new net N$52: JP1.5
- new net N$53: JP1.3
- new net N$54: JP1.1
- new net N$55: JP1.4
- new net N$56: JP2.8
- new net N$57: JP2.6
- new net N$58: JP2.4
- new net N$59: JP2.7
- new net N$60: JP2.9
- new net N$61: JP2.3
- new net N$62: JP2.5
- new net N$63: JP2.1
- new net N$65: R19.2, R23.1, T2.B
- new net PGND: D2.A, MD_GND.P, PAD12.P, P_GND1.P, SJGND.2, SJGND1.2, U$1.P$23, U$1.P$24, U$3.P$2
- new net RPI_GPIO17: SV1.11
- new net RPI_GPIO18: SV1.12
- new net RPI_GPIO22: SV1.15
- new net RPI_GPIO23: SV1.16
- new net RPI_GPIO24: SV1.18
- new net RPI_GPIO25: SV1.22
- new net RPI_GPIO27: SV1.13
- new net RPI_SPI0_CE0: SV1.24
- new net RPI_SPI0_CE1: SV1.26
- new net RPI_SPI0_MISO: SV1.21
- new net RPI_SPI0_MOSI: SV1.19
- new net RPI_SPI0_SCL: SV1.23
- new net RPI_VCC: J_RPIVCC.1, RTC.1, SV1.1, SV1.17
- new net UB_: C7.2, Q2.D, R25.1
- new net UCH: C6.2, Q2.S, R18.1, U$3.P$1
- net BUS_FON: now also BUS_1-3.S, P_BUS_FON.P; no longer PAD28.P, SV3.3
- net BUS_INT: now also BUS_1-9.S, P_BUS_INT.P; no longer PAD34.P, SV2.1, SV3.9
- net BUS_RESET: now also BUS_1-5.S, P_BUS_RESET.P; no longer PAD30.P, PAD40.P, SV2.5, SV3.5
- net BUS_SCL: now also BUS_1-7.S, P_BUS_SCL.P; no longer PAD32.P, PAD38.P, SV2.3, SV3.7
- net BUS_SDA: now also BUS_1-1.S, P_BUS_SDA.P; no longer PAD26.P, PAD36.P, PAD39.P, SV2.4, SV3.1
- net GND: now also BUS_1-10.S, BUS_1-8.S, C4.1, C5.2, DC_GND4.P, GPS2.2, JP1.6, JP2.10, JP2.2, OLED.1, P_GND2.P, R12.1, R13.1, R14.1, R15.1, SJGND1.1, SV5.7, U$2.1, U$4.1; no longer J_OLED3.1, J_OLED4.1, PAD33.P, PAD35.P, PAD41.P, SJ1.2, SV1.9, SV2.6, SV3.10, SV3.8
- net GNDA: now also C6.1, C7.1, DC_GND3.P, R19.1, SJGND.1, SV1.14, SV1.20, SV1.25, SV1.9, T2.E; no longer D2.A, MD_GND.P, PAD_GNDA.P, SJ1.1, U$1.P$23, U$1.P$24
- net ML_OUTA: now also P_ML_OUTA.P; no longer PAD_MLP.P
- net ML_OUTB: now also P_ML_OUTB.P; no longer PAD_MLR.P
- net MM_OUTA: now also P_MM_OUTA.P, U$3.P$24
- net MM_OUTB: now also P_MM_OUTB.P, U$3.P$23
- net MR_OUTA: now also P_MR_OUTA.P; no longer PAD_MRP.P
- net MR_OUTB: now also P_MR_OUTB.P; no longer PAD_MRN.P
- net OLED_SCL: now also OLED.3; no longer OLED1.3
- net OLED_SDA: now also OLED.4; no longer OLED1.4
- net RPI_RXD: now also SV1.10; no longer R1.2
- net RPI_TXD: now also SV1.8; no longer R2.2
- net SCL_SCK: now also SV5.6
- net SDA_MOSI: now also SV5.5
- net U55SW: now also BUS_1-4.S, P_U5SW.P, R.4, U$3.P$19
- net UB: now also J_UBSW1.1, R25.2; no longer R.5
- net UBSW: now also J_UBSW.1, P_UBSW.P, P_UBSW1.P, P_UBSW2.P; no longer DC_VIN1.P, PAD31.P, SV3.6
- net UBUS: now also BUS_1-2.S, P_UBUS.P; no longer PAD27.P, PAD37.P, SV2.2, SV3.2
- net VCC: now also OLED.2, R16.1, R17.1, VCC.P; no longer J_OLED3.3, J_OLED4.3
Other:
- note added: "(X)"
- note added: "3.3V DC/DC CONVERTER"
- note added: "3.3V Logic"
- note added: "5.5V DC/DC CONVERTER"
- note added: "Ardusimple ZED F9P"
- note added: "BNO055: accelerometer gyroscope magnetometer"
- note added: "simpleRTK2Blite"
- note removed: "DC/DC"
- moved on the sheet: L, PAD12, PAD13, PAD14, PAD15, PAD16, PAD17, PAD18, PAD19, PAD20, PAD21, PAD22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
