File: hw/rtk1010_test.brd (EAGLE design)
At the start: 36.8 x 20.3 mm, 19 parts

Commit message: rtk1010 board updated
Connections:
- net N$10 renamed VCC
- net N$12 renamed EN
- net N$13 renamed V_BKUP
- net N$2 renamed LNA_EN
- net N$3 renamed GPIO26
- net N$4 renamed TIMEPULSE
- net N$5 renamed RX
- net N$6 renamed TX
- net N$9 renamed RF_IN
Changed lines of the file:
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@@
 </elements>
 <signals>
-<signal name="N$2">
+<signal name="LNA_EN">
 <contactref element="LNA_EN" pad="1"/>
 <contactref element="U$1" pad="P$13"/>
@@
 <wire x1="18.7325" y1="6.35" x2="15.24" y2="6.35" width="0.6096" layer="16"/>
 </signal>
-<signal name="N$3">
+<signal name="GPIO26">
 <contactref element="GPIO26" pad="1"/>
 <contactref element="U$1" pad="P$18"/>
@@
 <wire x1="17.78" y1="5.08" x2="19.685" y2="5.08" width="0.6096" layer="16"/>
 </signal>
-<signal name="N$4">
+<signal name="TIMEPULSE">
 <contactref element="TIMEPULSE" pad="1"/>
 <contactref element="U$1" pad="P$4"/>
@@
 <wire x1="20.32" y1="3.4925" x2="20.32" y2="2.54" width="0.6096" layer="16"/>
 </signal>
-<signal name="N$5">
+<signal name="RX">
 <contactref element="RX" pad="1"/>
 <contactref element="U$1" pad="P$3"/>
@@
 <wire x1="30.98" y1="14.74" x2="33.02" y2="12.7" width="0.6096" layer="16"/>
 </signal>
-<signal name="N$6">
+<signal name="TX">
 <contactref element="TX" pad="1"/>
 <contactref element="U$1" pad="P$2"/>
@@
 <wire x1="32.42" y1="15.84" x2="33.02" y2="15.24" width="0.6096" layer="16"/>
 </signal>
-<signal name="N$9">
+<signal name="RF_IN">
 <contactref element="U$1" pad="P$11"/>
 <contactref element="L" pad="2"/>
@@
 <wire x1="13.335" y1="12.54" x2="13.335" y2="14.89" width="0.6096" layer="16"/>
 </signal>
-<signal name="N$10">
+<signal name="VCC">
 <contactref element="U$1" pad="P$8"/>
 <contactref element="R" pad="1"/>
@@
 <wire x1="33.02" y1="5.4" x2="32.7" y2="5.08" width="0.6096" layer="16"/>
 </signal>
-<signal name="N$12">
+<signal name="EN">
 <contactref element="U$1" pad="P$9"/>
 <contactref element="EN" pad="1"/>
@@
 <wire x1="25.66" y1="2.8" x2="25.4" y2="2.54" width="0.6096" layer="16"/>
 </signal>
-<signal name="N$13">
+<signal name="V_BKUP">
 <contactref element="V_BCKP" pad="1"/>
 <contactref element="U$1" pad="P$6"/>

Commit message: updated
Parts:
- moved PAD1 3.81 mm to (2.54, 11.4)
- moved PAD2 3.81 mm to (2.54, 6.35)
- moved PAD3 3.81 mm to (7.62, 6.35)
- moved PAD4 3.81 mm to (7.62, 11.4)
- moved L 3.81 mm to (11.4, 10.1)
- moved PAD5 3.81 mm to (5.08, 8.89)
- moved SJ1 0.71 mm to (29.9, 10.3)
Routing:
- net RF_IN: track 14.4 -> 11.0 mm
- net GND: track 92.4 -> 94.9 mm
- net N$8: track 6.75 -> 5.00 mm
- net VCC: track 9.30 -> 10.7 mm
- net V_BKUP: track 15.2 -> 15.7 mm
