File: hw/rtk1010_test.brd (EAGLE design)
At the start: 36.8 x 20.3 mm, 19 parts

Commit message: some optimiziations
Parts:
- removed PAD1, PAD2, PAD3, PAD4, PAD5: (no value), wirepad:3,17/1,3
- added C1: (no value), rcl:SMC_B
- added J2: J_SMA_TYCO_1053378, j_sma_tyco_1053378-1:1053378-1
Connections:
- net GND: now also C1.-, J2.GND_1, J2.GND_2, J2.GND_3, J2.GND_4; no longer PAD1.1, PAD2.1, PAD3.1, PAD4.1
- net RF_IN: now also J2.ANT; no longer PAD5.1
- net VCC: now also C1.+
Routing:
- net GND: track 94.9 -> 92.1 mm, vias 0 -> 13
- added copper zone on layer 1, net GND
Other:
- outline, holes or cut-outs redrawn
