File: hw/rtk1010_test.sch (EAGLE design)
At the start: 19 parts

Commit message: rtk1010 board updated
Connections:
- net N$10 renamed VCC
- net N$12 renamed EN
- net N$13 renamed V_BKUP
- net N$2 renamed LNA_EN
- net N$3 renamed GPIO26
- net N$4 renamed TIMEPULSE
- net N$5 renamed RX
- net N$6 renamed TX
- net N$9 renamed RF_IN
Changed lines of the file:
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@@
 </segment>
 </net>
-<net name="N$2" class="0">
+<net name="LNA_EN" class="0">
 <segment>
 <pinref part="LNA_EN" gate="1" pin="P"/>
@@
 </segment>
 </net>
-<net name="N$3" class="0">
+<net name="GPIO26" class="0">
 <segment>
 <pinref part="GPIO26" gate="1" pin="P"/>
@@
 </segment>
 </net>
-<net name="N$4" class="0">
+<net name="TIMEPULSE" class="0">
 <segment>
 <pinref part="TIMEPULSE" gate="1" pin="P"/>
@@
 </segment>
 </net>
-<net name="N$5" class="0">
+<net name="RX" class="0">
 <segment>
 <pinref part="RX" gate="1" pin="P"/>
@@
 </segment>
 </net>
-<net name="N$6" class="0">
+<net name="TX" class="0">
 <segment>
 <pinref part="TX" gate="1" pin="P"/>
@@
 </segment>
 </net>
-<net name="N$9" class="0">
+<net name="RF_IN" class="0">
 <segment>
 <pinref part="U$1" gate="G$1" pin="RF_IN"/>
@@
 </segment>
 </net>
-<net name="N$10" class="0">
+<net name="VCC" class="0">
 <segment>
 <pinref part="U$1" gate="G$1" pin="VCC"/>
@@
 </segment>
 </net>
-<net name="N$12" class="0">
+<net name="EN" class="0">
 <segment>
 <pinref part="U$1" gate="G$1" pin="EN"/>
@@
 </segment>
 </net>
-<net name="N$13" class="0">
+<net name="V_BKUP" class="0">
 <segment>
 <pinref part="V_BCKP" gate="1" pin="P"/>

Commit message: some optimiziations
Parts:
- removed PAD1, PAD2, PAD3, PAD4, PAD5: (no value), wirepad:3,17/1,3
- added C1: (no value), rcl:CPOL-EUSMCB
- added J2: J_SMA_TYCO_1053378, j_sma_tyco_1053378-1:J_SMA_TYCO_1053378
Connections:
- net GND: now also C1.-, J2.RFGND_1, J2.RFGND_2, J2.RFGND_3, J2.RFGND_4; no longer PAD1.P, PAD2.P, PAD3.P, PAD4.P
- net RF_IN: now also J2.RF_IN; no longer PAD5.P
- net VCC: now also C1.+
Other:
- moved on the sheet: EN, R, VCC
