File: kicad/IndegoMower/processor.kicad_sch (KiCad schematic)
At the start: 1 part

Commit message: -
Parts:
- U7: value (none) -> ATmega128A-A; footprint (none) -> Package_QFP:TQFP-64_14x14mm_P0.8mm
Changed lines of the file:
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@@
       (effects (font (size 1.27 1.27)) (justify left))
     )
-    (property "Value" "" (id 1) (at 112.5094 143.51 0)
+    (property "Value" "ATmega128A-A" (id 1) (at 112.5094 143.51 0)
       (effects (font (size 1.27 1.27)) (justify left))
     )
-    (property "Footprint" "" (id 2) (at 110.49 90.17 0)
+    (property "Footprint" "Package_QFP:TQFP-64_14x14mm_P0.8mm" (id 2) (at 110.49 90.17 0)
       (effects (font (size 1.27 1.27) italic) hide)
     )
@@
   (symbol (lib_id "power:VCC") (at 110.49 39.37 0) (unit 1)
     (in_bom yes) (on_board yes) (fields_autoplaced)
-    (property "Reference" "#PWR0114" (id 0) (at 110.49 43.18 0)
+    (property "Reference" "#PWR0113" (id 0) (at 110.49 43.18 0)
       (effects (font (size 1.27 1.27)) hide)
     )
-    (property "Value" "" (id 1) (at 110.49 34.29 0))
+    (property "Value" "VCC" (id 1) (at 110.49 34.29 0))
     (property "Footprint" "" (id 2) (at 110.49 39.37 0)
       (effects (font (size 1.27 1.27)) hide)
@@
   (symbol (lib_id "power:GNDD") (at 110.49 140.97 0) (unit 1)
     (in_bom yes) (on_board yes) (fields_autoplaced)
-    (property "Reference" "#PWR0113" (id 0) (at 110.49 147.32 0)
+    (property "Reference" "#PWR0114" (id 0) (at 110.49 147.32 0)
       (effects (font (size 1.27 1.27)) hide)
     )
-    (property "Value" "" (id 1) (at 110.49 146.05 0))
+    (property "Value" "GNDD" (id 1) (at 110.49 146.05 0))
     (property "Footprint" "" (id 2) (at 110.49 140.97 0)
       (effects (font (size 1.27 1.27)) hide)
