File: kicad/IndegoMower/rpi.kicad_sch (KiCad schematic)
At the start: 1 part

Commit message: -
Parts:
- J1: value (none) -> RPi_GPIO; footprint (none) -> Connector_PinSocket_2.54mm:PinSocket_2x20_P2.54mm_Vertical_SMD
Changed lines of the file:
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@@
       (effects (font (size 1.27 1.27)) hide)
     )
-    (property "Value" "" (id 1) (at 153.543 125.73 0))
+    (property "Value" "GNDPWR" (id 1) (at 153.543 125.73 0))
     (property "Footprint" "" (id 2) (at 153.67 121.92 0)
       (effects (font (size 1.27 1.27)) hide)
@@
       (effects (font (size 1.524 1.524)))
     )
-    (property "Value" "" (id 1) (at 128.27 63.5 0)
+    (property "Value" "RPi_GPIO" (id 1) (at 128.27 63.5 0)
       (effects (font (size 1.524 1.524)))
     )
-    (property "Footprint" "" (id 2) (at 109.22 67.31 0)
+    (property "Footprint" "Connector_PinSocket_2.54mm:PinSocket_2x20_P2.54mm_Vertical_SMD" (id 2) (at 109.22 67.31 0)
       (effects (font (size 1.524 1.524)))
     )
