File: kicad/IndegoMower/IndegoMower.kicad_pcb (KiCad board)
At the start: 2 copper layers, 170 x 230 mm, 145 parts, among them J1 RPi_GPIO, Q1 BC847, Q2 TSM480P06CP, Q3 BC847, U1 26SHC-B-1A, U2 24SHC-B-1A, U3 LM2596S-ADJ, U4 LM317_TO-252, U7 ATmega128A-A

Commit message: some more work
Parts:
- added C3: ~, Capacitor_SMD:C_0805_2012Metric_Pad1.18x1.45mm_HandSolder, B.Cu at (95.2, 154.9)
- added C4: ~, Capacitor_SMD:CP_Elec_16x17.5, B.Cu at (87.7, 144.8)
- added C5: ~, Capacitor_SMD:CP_Elec_16x17.5, B.Cu at (87.7, 179.1)
- added C6: ~, Capacitor_SMD:C_0805_2012Metric_Pad1.18x1.45mm_HandSolder, F.Cu at (80.0, 151.1)
- added C8: ~, Capacitor_SMD:C_0805_2012Metric_Pad1.18x1.45mm_HandSolder, B.Cu at (95.2, 168.9)
- added D16: ~, Diode_SMD:D_SMA-SMB_Universal_Handsoldering, F.Cu at (88.9, 154.9)
- added JP2: ~, Jumper:SolderJumper-2_P1.3mm_Open_RoundedPad1.0x1.5mm, F.Cu at (297.7, 135.2)
- added J_U55_GND3: ~, Connector_Wire:SolderWire-1sqmm_1x01_D1.4mm_OD2.7mm, F.Cu at (78.7, 142.2)
- added J_U55_GND4: ~, Connector_Wire:SolderWire-1sqmm_1x01_D1.4mm_OD2.7mm, F.Cu at (78.7, 181.6)
- added J_U55_IN2: ~, Connector_Wire:SolderWire-1sqmm_1x01_D1.4mm_OD2.7mm, F.Cu at (96.5, 142.2)
- added J_U55_OUT2: ~, Connector_Wire:SolderWire-1sqmm_1x01_D1.4mm_OD2.7mm, F.Cu at (96.5, 181.6)
- added J_UM_ON3: ~, Connector_Wire:SolderWire-1sqmm_1x01_D1.4mm_OD2.7mm, F.Cu at (292.9, 128.1)
- added L4: 33uH, Inductor_SMD:L_Fastron_PISR_Handsoldering, B.Cu at (87.1, 162.6)
- added Q6: ~, Package_TO_SOT_SMD:SOT-23_Handsoldering, F.Cu at (283.9, 134.4)
- added R27: ~, Resistor_SMD:R_0805_2012Metric_Pad1.20x1.40mm_HandSolder, F.Cu at (291.5, 131.9)
- added R28: ~, Resistor_SMD:R_0805_2012Metric_Pad1.20x1.40mm_HandSolder, F.Cu at (80.0, 153.7)
- added R29: ~, Resistor_SMD:R_0805_2012Metric_Pad1.20x1.40mm_HandSolder, F.Cu at (80.0, 156.2)
- added R7: ~, Resistor_SMD:R_0805_2012Metric_Pad1.20x1.40mm_HandSolder, F.Cu at (292.7, 136.8)
- added R8: ~, Resistor_SMD:R_0805_2012Metric_Pad1.20x1.40mm_HandSolder, F.Cu at (293.4, 139.7)
- added U8: ~, Package_TO_SOT_SMD:TO-263-5_TabPin3, F.Cu at (84.1, 166.7)
- moved C18 1.27 mm to (70.9, 168.9)
Routing:
- net GNDPWR: track 296.7 -> 291.6 mm
