File: kicad/IndegoMower/IndegoMower.kicad_sch (KiCad schematic)
At the start: 0 parts

Commit message: some more work
Other:
- added sheet ESP32 (esp32.kicad_sch)
- added sheet Extension Bus (extension_bus.kicad_sch)
- added sheet GPS (gps.kicad_sch)
- added sheet IMU (imu.kicad_sch)
- note added: "* AVR Mega128"
- note added: "* BNO055 IMU"
- note added: "* Connectors * Sensors * Bat Charger * Indego UI (Button + LCD) * STOP Button"
- note added: "* ESP32-S2/S3 * SDCard * Camera (OV2640)"
- note added: "* I2C Bus * SPI Bus"
- note added: "* LM2596HVS DC/DC"
- note added: "* RPI 3/4 * RPI Zero 2W * Banana PI Zero M2"
- note added: "* VNH 3SP30 H Bridge"
- note added: "* simpleRTK2B Lite * RTK-1010 * GPS Antenna * LNA"
- note added: "Architecture: * should work with Indego 1000, 1200 and 1300 * fit to origional ALM mainboard dimensions * support for all Indego Sensors * AVR MeGa 128 used for low power/standby uC * ESP32 S3 for connected processor (microROS) * RPI4 or compatibe linux/SBC (optional) * RTK GPS (Ublox F9P or RTK-1010) * onboard GPS L1/L2 antenna (LNA?) * use low cost modules/parts much as possible (DC/DC converte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"
