File: kicad/IndegoMower/powersupply.kicad_sch (KiCad schematic)
At the start: 79 parts, among them Q1 BC847, Q2 TSM480P06CP, Q3 BC847, U3 LM2596S-ADJ, U4 LM317_TO-252

Commit message: some more work
Parts:
- removed JP3: ~, Jumper:SolderJumper-2_P1.3mm_Open_RoundedPad1.0x1.5mm, symbol Jumper:SolderJumper_2_Open
- removed J_B10, J_B11, J_B12, J_B9: ~, Connector_Wire:SolderWire-1sqmm_1x01_D1.4mm_OD2.7mm, symbol Connector:Conn_01x01_Female
- removed U4: LM317_TO-252, Package_TO_SOT_SMD:TO-252-2, symbol Regulator_Linear:LM317_TO-252
- added D16: (no value), symbol Diode:MBRA340
- added J_U55_GND3, J_U55_GND4, J_U55_IN2, J_U55_OUT2, J_UM_ON3: (no value), symbol Connector:Conn_01x01_Female
- added L4: (no value), symbol Device:L
- added Q6: (no value), symbol Transistor_BJT:BC847
- added R27, R28, R29: (no value), symbol Device:R
- added U10: ~, symbol Regulator_Linear:LM1117-3.3
- added U4: ~, symbol 2022-05-19_16-24-53:max5084att+t
- added U8: (no value), symbol Regulator_Switching:LM2596S-ADJ
- added U9: ~, symbol Regulator_Linear:MCP1703A-5002_SOT89
- C3, C6, C8: value 0.1 -> (none); footprint Capacitor_SMD:C_0805_2012Metric_Pad1.18x1.45mm_HandSolder -> (none)
- C4, C5: value ~ -> (none); footprint Capacitor_SMD:CP_Elec_16x17.5 -> (none)
- JP2: value SolderJumper_2_Open -> (none); footprint Jumper:SolderJumper-2_P1.3mm_Open_RoundedPad1.0x1.5mm -> (none)
- R7, R8: value ~ -> (none); footprint Resistor_SMD:R_0805_2012Metric_Pad1.20x1.40mm_HandSolder -> (none)
Connections:
- net GNDPWR: now also D16.2 (A), J_U55_GND3.1 (Pin_1), J_U55_GND4.1 (Pin_1), Q6.2 (E), R29.2, U8.3 (GND); no longer C6.2
- net ON_U24: now also R7.2
- net UB: no longer C3.1, C4.1
- net U_55: now also C5.1, C6.2, C8.1, J_U55_OUT2.1 (Pin_1), L4.2, R28.1
- net U_BAT_SW: now also C3.1, C4.1, J_U55_IN2.1 (Pin_1), R27.1, U8.1 (VIN)
- net at JP2.1 (A), R7.1: now also R8.1, Q6.1 (B); no longer C5.1, C6.1
- net VCC: no longer names the net of JP2.2 (B)
- net VCC: now also J_UM_ON3.1 (Pin_1), Q6.3 (C), R27.2, U8.5 (~{ON}/OFF); no longer C8.1
- new net: D16.1 (K), L4.1, U8.2 (OUT)
- new net: C6.1, R28.2, R29.1, U8.4 (FB)
Other:
- note added: "Main CPU (RPI) Power Supply (5.5V,3A)"
- note added: "Standby Power Supply (3.3V, 50mA, low Iq)"
- note added: "VCC Power Supply (5V,3A)"
- note removed: "Main CPU Power Supply (12V,3A)"
- note removed: "Main CPU Power Supply (5.5V,3A)"
- note removed: "Standby Power Supply (3.3V,1.5A, low Iq)"
- note removed: "optional MP1584EN"
