File: kicad/MainPCB/processor.kicad_sch (KiCad schematic)
At the start: 1 part, among them U10 ATmega128A-A

Commit message: some further progress
Parts:
- added U17: ATtiny3216-S, Package_SO:SOIC-20W_7.5x12.8mm_P1.27mm, symbol MCU_Microchip_ATtiny:ATtiny3216-S
Changed lines of the file:
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@@
+	)
+	(symbol
+		(lib_id "MCU_Microchip_ATtiny:ATtiny3216-S")
+		(at 196.85 76.2 0)
+		(unit 1)
+		(exclude_from_sim no)
+		(in_bom yes)
+		(on_board yes)
+		(dnp no)
+		(fields_autoplaced yes)
+		(property "Reference" "U17"
+			(at 198.9933 50.8 0)
+			(effects
+				(font
+					(size 1.27 1.27)
+				)
+				(justify left)
+			)
+		)
+		(property "Value" "ATtiny3216-S"
+			(at 198.9933 53.34 0)
+			(effects
+				(font
+					(size 1.27 1.27)
+				)
+				(justify left)
+			)
+		)
+		(property "Footprint" "Package_SO:SOIC-20W_7.5x12.8mm_P1.27mm"
+			(at 196.85 76.2 0)
+			(effects
+				(font
+					(size 1.27 1.27)
+					(italic yes)
+				)
+				(hide yes)
+			)
+		)
+		(property "Datasheet" "http://ww1.microchip.com/downloads/en/DeviceDoc/ATtiny3216_ATtiny1616-data-sheet-40001997B.pdf"
+			(at 196.85 76.2 0)
+			(effects
+				(font
+					(size 1.27 1.27)
+				)
+				(hide yes)
+			)
+		)
+		(property "Description" "20MHz, 32kB Flash, 2kB SRAM, 256B EEPROM, SOIC-20"
+			(at 196.85 76.2 0)
+			(effects
+				(font
+					(size 1.27 1.27)
+				)
+				(hide yes)
+			)
+		)
+		(pin "1"
+		)
+		(pin "20"
+		)
+		(pin "5"
+		)
+		(pin "4"
+		)
+		(pin "11"
+		)
+		(pin "7"
+		)
+		(pin "18"
+		)
+		(pin "15"
+		)
+		(pin "9"
+		)
+		(pin "14"
+		)
+		(pin "16"
+		)
+		(pin "13"
+		)
+		(pin "8"
+		)
+		(pin "12"
+		)
+		(pin "3"
+		)
+		(pin "6"
+		)
+		(pin "10"
+		)
+		(pin "2"
+		)
+		(pin "17"
+		)
+		(pin "19"
+		)
+		(instances
+			(project ""
+				(path "/9538e4ed-27e6-4c37-b989-9859dc0d49e8/779e8a7f-993e-44a7-9f1f-511b922b345b"
+					(reference "U17")
+					(unit 1)
+				)
+			)
+		)
 	)
 	(symbol
