File: kicad/MainPCB/IndegoMower.kicad_pcb (KiCad board)
At the start: 2 copper layers, 172 x 230 mm, 223 parts, among them J1 RPi_GPIO, J9 RPi_GPIO, Q1 BC847, Q10 BC817, Q11 BC817, Q2 TSM480P06CP, Q3 BC847, Q7 BC817, Q8 BC817, Q9 BC817, U1 26SHC-B-1A, U10 ATmega128A-A, U11 TCA9800, U12 MAX11617, U13 MCP23017_SS, U14 ESP32-S3-WROOM-2 (-1), U15 XC6206-2.8V, U16 RT9166-12GVL, U17 ATtiny3216-S, U18 L298P, U2 24SHC-B-1A, U4 LM2596S-ADJ

Commit message: ...
Parts:
- removed C1, C14, C21, C22, C45, C46, C47, C48: 0.1, Capacitor_SMD:C_0805_2012Metric_Pad1.18x1.45mm_HandSolder
- removed C10, C11, C12, C6, C7, C8: ~, Capacitor_SMD:CP_Elec_16x17.5
- removed C13: 560pF, Capacitor_SMD:C_0805_2012Metric_Pad1.18x1.45mm_HandSolder
- removed C15, C16, C17, C18, C19, C2, C20, C23, C3, C4: ~, Capacitor_SMD:C_0805_2012Metric_Pad1.18x1.45mm_HandSolder
- removed C29, C30, C31, C32, C33, C34, C36, C37, C38, C39, C44: 10u_0402_CL05A105KA5NQNC, Capacitor_SMD:C_0402_1005Metric
- removed C35: 22p_0402_0402CG220J500NT, Capacitor_SMD:C_0402_1005Metric
- removed C5: 680uF/50V, Capacitor_SMD:CP_Elec_16x17.5
- removed C9: 220uF/40V, Capacitor_SMD:CP_Elec_16x17.5
- removed D1, D2, D3, D4: ~, Diode_SMD:D_SMA-SMB_Universal_Handsoldering
- removed D13, D14, D15, D16, D23, D24, D25, D26, D27, D28, D29, D30: ~, Diode_SMD:D_SMA_Handsoldering
- removed D17, D18, D20, D21, D22: SOD-523_BSD5C051L, Diode_SMD:D_SOD-523
- removed D19: 1N4148W, Diode_SMD:D_SOD-123
- removed D6, D7: SM6T30A, Diode_SMD:D_SMB
- removed J9: RPi_GPIO, RPI_Hat:RPI_Hat_B+
- removed JP1: SolderJumper_2_Open, Jumper:SolderJumper-2_P1.3mm_Open_RoundedPad1.0x1.5mm
- removed JP2, JP3, JP4: ~, Jumper:SolderJumper-2_P1.3mm_Open_RoundedPad1.0x1.5mm
- removed J_B1, J_B2, J_B3, J_B4, J_B5, J_B6, J_B7: ~, Connector_Wire:SolderWire-0.5sqmm_1x01_D0.9mm_OD2.1mm
- removed J_MM_GND1, J_MM_OUTA1, J_MM_OUTB1, J_MM_VCC1, J_U55_GND1, J_U55_GND2, J_U55_GND3, J_U55_GND4, J_U55_IN1, J_U55_IN2, J_U55_OUT1, J_U55_OUT2, J_UD_GND1, J_UD_GND2, J_UD_IN1, J_UD_ON1, J_UD_OUT1, J_UM_GND1, J_UM_GND2, J_UM_IN1, J_UM_ON1, J_UM_ON2, J_UM_ON3, J_UM_OUT1: ~, Connector_Wire:SolderWire-1sqmm_1x01_D1.4mm_OD2.7mm
- removed L1, L2, L3, L4: 33uH, Inductor_SMD:L_Fastron_PISR_Handsoldering
- removed L5: FB_2A_0805_220R@100MHz_BLM21PG221SN1D, Inductor_SMD:L_0805_2012Metric_Pad1.15x1.40mm_HandSolder
- removed Q1: BC847, Package_TO_SOT_SMD:SOT-23
- removed Q10, Q11, Q7, Q8, Q9: BC817, Package_TO_SOT_SMD:SOT-23
- removed Q2: TSM480P06CP, Package_TO_SOT_SMD:TO-252-2
- removed Q3: BC847, Package_TO_SOT_SMD:SOT-23_Handsoldering
- removed Q4, Q5, Q6: ~, Package_TO_SOT_SMD:SOT-23_Handsoldering
- removed R1, R4: 10k, Resistor_SMD:R_0805_2012Metric_Pad1.20x1.40mm_HandSolder
- removed R10, R11, R13, R14, R15, R16, R17, R18, R19, R20, R21, R22, R23, R28, R29, R5, R6, R7, R9: ~, Resistor_SMD:R_0805_2012Metric_Pad1.20x1.40mm_HandSolder
- removed R12: 100k, Resistor_SMD:R_0805_2012Metric_Pad1.20x1.40mm_HandSolder
- removed R2, R8: 47k, Resistor_SMD:R_0805_2012Metric_Pad1.20x1.40mm_HandSolder
- removed R24, R68: 0.01, Resistor_SMD:R_0805_2012Metric_Pad1.20x1.40mm_HandSolder
- removed R25, R69, R70, R71, R72, R73, R74, R75, R76, R77, R78, R79, R80, R81: 1k, Resistor_SMD:R_0805_2012Metric_Pad1.20x1.40mm_HandSolder
- removed R26, R27, R30, R31, R34, R40, R41, R44, R48, R49, R50, R51, R52, R53, R54, R55, R56, R61, R64, R67, R82, R83, R84, R85, R86, R87: 10k, Resistor_SMD:R_0805_2012Metric
- removed R3: 330k, Resistor_SMD:R_0805_2012Metric_Pad1.20x1.40mm_HandSolder
- removed R32, R33, R35: 22, Resistor_SMD:R_0805_2012Metric
- removed R36, R37, R38, R39, R42, R43, R45, R46, R47: 100, Resistor_SMD:R_0805_2012Metric
- removed R57, R60, R63, R66: 100k, Resistor_SMD:R_0805_2012Metric
- removed R58, R59, R62, R65: n.b., Resistor_SMD:R_0805_2012Metric
- removed U10: ATmega128A-A, Package_QFP:TQFP-64_14x14mm_P0.8mm
- removed U11: TCA9800, Package_SO:VSSOP-8_3x3mm_P0.65mm
- removed U12: MAX11617, Package_SO:QSOP-16_3.9x4.9mm_P0.635mm
- removed U13: MCP23017_SS, Package_SO:SSOP-28_5.3x10.2mm_P0.65mm
- removed U15: XC6206-2.8V, Package_TO_SOT_SMD:SOT-23
- removed U16: RT9166-12GVL, Package_TO_SOT_SMD:SOT-23
- removed U17: ATtiny3216-S, Package_SO:SOIC-20W_7.5x12.8mm_P1.27mm
- removed U4: LM2596S-ADJ, Package_TO_SOT_SMD:TO-263-5_TabPin3
- removed U5, U6, U7: ~, Package_TO_SOT_SMD:TO-263-5_TabPin3
- added REF**: MountingHole_3.2mm_M3, MountingHole:MountingHole_3.2mm_M3, F.Cu at (109.0, 78.0)
- added REF**: MountingHole_3.2mm_M3, MountingHole:MountingHole_3.2mm_M3, F.Cu at (85.0, 54.0)
- added REF**: MountingHole_3.2mm_M3, MountingHole:MountingHole_3.2mm_M3, F.Cu at (85.0, 78.0)
- added REF**: MountingHole_3.2mm_M3, MountingHole:MountingHole_3.2mm_M3, F.Cu at (109.0, 54.0)
- J1: footprint Connector_PinSocket_2.54mm:PinSocket_2x20_P2.54mm_Vertical_SMD -> Connector_PinSocket_2.54mm:PinSocket_2x20_P2.54mm_Vertical; moved to B.Cu
- moved J_MM1 311.9 mm to (188.0, 127.0)
- moved F_SEC1 262.9 mm to (45.7, 109.5), turned to -90 degrees
- moved J1 258.5 mm to (114.3, 31.9), turned to 180 degrees
- moved F_MAIN1 249.5 mm to (35.6, 109.5), turned to -90 degrees
- moved F_CHARGE1 233.7 mm to (33.3, 154.9)
- moved U18 175.6 mm to (49.0, 55.9)
- moved U14 12.6 mm to (176.1, 36.7), turned to -45 degrees
Connections:
- U1 pad P$24: GNDPWR -> Net-(U1-P$23)
- U1 pad P$25: GNDPWR -> Net-(U1-P$23)
- U18 pad 16: MR_N -> MR_P
Routing:
- net GNDPWR: track 0.00 -> 224.4 mm
- net MR_P: track 0.00 -> 25.5 mm
- net MR_N: track 0.00 -> 25.1 mm
- net ML_N: track 0.00 -> 23.4 mm
- net ML_P: track 0.00 -> 23.3 mm
- net Net-(U1-P$25): track 0.00 -> 13.8 mm
- net Net-(U2-P$1): track 0.00 -> 13.6 mm
- net UB: track 0.00 -> 10.2 mm
- net Net-(U1-P$26): track 0.00 -> 9.87 mm
Other:
- outline, holes or cut-outs redrawn
- board text added: "free"
