File: kicad/MainPCB/rpi.kicad_sch (KiCad schematic)
At the start: 1 part, among them J1 RPi_GPIO

Commit message: ...
Parts:
- added J9: RPi_GPIO, Connector_PinSocket_2.54mm:PinSocket_2x20_P2.54mm_Vertical, symbol RPi_Hat:RPi_GPIO
- J1: footprint Connector_PinSocket_2.54mm:PinSocket_2x20_P2.54mm_Vertical_SMD -> Connector_PinSocket_2.54mm:PinSocket_2x20_P2.54mm_Vertical
Connections:
- net GNDPWR: now also J9.14 (GND), J9.20 (GND), J9.25 (GND), J9.30 (GND), J9.34 (GND), J9.39 (GND), J9.6 (GND), J9.9 (GND)
- net U_55: now also J9.2 (5V), J9.4 (5V)
